File: pdb.sch (EAGLE design)
At the start: 49 parts, among them Q1 20MHz, Q2 IRFR5305PBF, Q3 IRFR5305PBF, U1 TSR_1-2433, U2 LTC2946CMSPBF, U3 LTC2946CMSPBF, U4 LTC2946CMSPBF, U5 ATMEGA48-20AU, U6 TXB0104, U7 AT30TS74SS8M

Commit message: sachen gemacht dass fusion glücklich ist
Parts:
- removed ISP: (no value), con-harting-ml:ML6
- added JP11: (no value), pinhead:PINHD-2X3/90
Connections:
- net +5V: now also JP11.2; no longer ISP.2
- net GND: now also JP11.6; no longer ISP.6
- net MISO_5V: now also JP11.1; no longer ISP.1
- net MOSI_5V: now also JP11.4; no longer ISP.4
- net RESET: now also JP11.5; no longer ISP.5
- net SCK_5V: now also JP11.3; no longer ISP.3
Changed lines of the file:
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@@
 <?xml version="1.0" encoding="utf-8"?>
 <!DOCTYPE eagle SYSTEM "eagle.dtd">
-<eagle version="8.6.2">
+<eagle version="8.6.3">
 <drawing>
 <settings>
@@
 <part name="R8" library="rcl" library_urn="urn:adsk.eagle:library:334" deviceset="R-EU_" device="R0805" package3d_urn="urn:adsk.eagle:package:23553/2" value="4,7k"/>
 <part name="R9" library="rcl" library_urn="urn:adsk.eagle:library:334" deviceset="R-EU_" device="R0805" package3d_urn="urn:adsk.eagle:package:23553/2" value="4,7k"/>
-<part name="ISP" library="con-harting-ml" library_urn="urn:adsk.eagle:library:149" deviceset="ML6" device="" package3d_urn="urn:adsk.eagle:package:6988/1"/>
 <part name="GND22" library="supply1" library_urn="urn:adsk.eagle:library:371" deviceset="GND" device=""/>
 <part name="SUPPLY21" library="supply2" deviceset="+5V" device=""/>
@@
 <part name="SJ1" library="jumper" library_urn="urn:adsk.eagle:library:252" deviceset="SJ" device="" package3d_urn="urn:adsk.eagle:package:15471/1"/>
 <part name="+3V4" library="supply1" library_urn="urn:adsk.eagle:library:371" deviceset="+3V3" device=""/>
+<part name="JP11" library="pinhead" library_urn="urn:adsk.eagle:library:325" deviceset="PINHD-2X3" device="/90" package3d_urn="urn:adsk.eagle:package:22464/2"/>
 </parts>
 <sheets>
@@
 <instance part="R8" gate="G$1" x="66.04" y="83.82" rot="R180"/>
 <instance part="R9" gate="G$1" x="66.04" y="91.44" rot="R180"/>
-<instance part="ISP" gate="1" x="208.28" y="78.74"/>
 <instance part="GND22" gate="1" x="185.42" y="73.66"/>
 <instance part="SUPPLY21" gate="+5V" x="193.04" y="76.2" rot="R90"/>
+<instance part="JP11" gate="A" x="208.28" y="78.74" rot="R180"/>
 </instances>
 <busses>
@@
 <pinref part="GND22" gate="1" pin="GND"/>
 <wire x1="185.42" y1="76.2" x2="185.42" y2="81.28" width="0.1524" layer="91"/>
-<pinref part="ISP" gate="1" pin="6"/>
-<wire x1="185.42" y1="81.28" x2="200.66" y2="81.28" width="0.1524" layer="91"/>
+<wire x1="185.42" y1="81.28" x2="203.2" y2="81.28" width="0.1524" layer="91"/>
+<pinref part="JP11" gate="A" pin="6"/>
 </segment>
 </net>
@@
 <segment>
 <pinref part="SUPPLY21" gate="+5V" pin="+5V"/>
-<pinref part="ISP" gate="1" pin="2"/>
-<wire x1="195.58" y1="76.2" x2="200.66" y2="76.2" width="0.1524" layer="91"/>
+<pinref part="JP11" gate="A" pin="2"/>
+<wire x1="195.58" y1="76.2" x2="203.2" y2="76.2" width="0.1524" layer="91"/>
 </segment>
 </net>
@@
 </segment>
 <segment>
-<pinref part="ISP" gate="1" pin="3"/>
 <wire x1="215.9" y1="78.74" x2="218.44" y2="78.74" width="0.1524" layer="91"/>
 <label x="218.44" y="78.74" size="1.016" layer="95" xref="yes"/>
+<pinref part="JP11" gate="A" pin="3"/>
+<wire x1="215.9" y1="78.74" x2="210.82" y2="78.74" width="0.1524" layer="91"/>
 </segment>
 </net>
@@
 </segment>
 <segment>
-<pinref part="ISP" gate="1" pin="5"/>
-<wire x1="215.9" y1="81.28" x2="218.44" y2="81.28" width="0.1524" layer="91"/>
 <label x="218.44" y="81.28" size="1.016" layer="95" xref="yes"/>
+<wire x1="218.44" y1="81.28" x2="210.82" y2="81.28" width="0.1524" layer="91"/>
+<pinref part="JP11" gate="A" pin="5"/>
 </segment>
 </net>
@@
 </segment>
 <segment>
-<pinref part="ISP" gate="1" pin="4"/>
-<wire x1="200.66" y1="78.74" x2="198.12" y2="78.74" width="0.1524" layer="91"/>
 <label x="198.12" y="78.74" size="1.016" layer="95" rot="R180" xref="yes"/>
+<pinref part="JP11" gate="A" pin="4"/>
+<wire x1="198.12" y1="78.74" x2="203.2" y2="78.74" width="0.1524" layer="91"/>
 </segment>
 </net>
@@
 </segment>
 <segment>
-<pinref part="ISP" gate="1" pin="1"/>
-<wire x1="215.9" y1="76.2" x2="218.44" y2="76.2" width="0.1524" layer="91"/>
 <label x="218.44" y="76.2" size="1.016" layer="95" xref="yes"/>
-</segment>
-</net>
+<pinref part="JP11" gate="A" pin="1"/>
+<wire x1="218.44" y1="76.2" x2="210.82" y2="76.2" width="0.1524" layer="91"/>
+</segment>
+</net>

Commit message: layout stuff
Parts:
- removed JP10, JP2, JP3, JP4, JP5, JP6, JP7, JP8, JP9: (no value), pinhead:PINHD-1X2
Connections:
- net +3V3: no longer JP10.1, JP8.1, JP9.1
- net +5V: no longer JP5.1, JP6.1, JP7.1
- net GND: no longer JP10.2, JP2.2, JP3.2, JP4.2, JP5.2, JP6.2, JP7.2, JP8.2, JP9.2
- net V+: no longer JP2.1, JP3.1, JP4.1
Changed lines of the file:
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@@
 <part name="SUPPLY21" library="supply2" deviceset="+5V" device=""/>
 <part name="R6" library="jonas_bourns" library_urn="urn:adsk.eagle:library:1422904" deviceset="CRA2512-FZ-R040ELF" device="" package3d_urn="urn:adsk.eagle:package:1633525/2"/>
-<part name="JP2" library="pinhead" library_urn="urn:adsk.eagle:library:325" deviceset="PINHD-1X2" device="" package3d_urn="urn:adsk.eagle:package:22435/2"/>
-<part name="JP3" library="pinhead" library_urn="urn:adsk.eagle:library:325" deviceset="PINHD-1X2" device="" package3d_urn="urn:adsk.eagle:package:22435/2"/>
-<part name="JP4" library="pinhead" library_urn="urn:adsk.eagle:library:325" deviceset="PINHD-1X2" device="" package3d_urn="urn:adsk.eagle:package:22435/2"/>
-<part name="SUPPLY20" library="supply2" library_urn="urn:adsk.eagle:library:372" deviceset="V+" device=""/>
-<part name="GND23" library="supply1" deviceset="GND" device=""/>
-<part name="JP5" library="pinhead" library_urn="urn:adsk.eagle:library:325" deviceset="PINHD-1X2" device="" package3d_urn="urn:adsk.eagle:package:22435/2"/>
-<part name="JP6" library="pinhead" library_urn="urn:adsk.eagle:library:325" deviceset="PINHD-1X2" device="" package3d_urn="urn:adsk.eagle:package:22435/2"/>
-<part name="JP7" library="pinhead" library_urn="urn:adsk.eagle:library:325" deviceset="PINHD-1X2" device="" package3d_urn="urn:adsk.eagle:package:22435/2"/>
-<part name="GND24" library="supply1" deviceset="GND" device=""/>
-<part name="JP8" library="pinhead" library_urn="urn:adsk.eagle:library:325" deviceset="PINHD-1X2" device="" package3d_urn="urn:adsk.eagle:package:22435/2"/>
-<part name="JP9" library="pinhead" library_urn="urn:adsk.eagle:library:325" deviceset="PINHD-1X2" device="" package3d_urn="urn:adsk.eagle:package:22435/2"/>
-<part name="JP10" library="pinhead" library_urn="urn:adsk.eagle:library:325" deviceset="PINHD-1X2" device="" package3d_urn="urn:adsk.eagle:package:22435/2"/>
-<part name="GND26" library="supply1" deviceset="GND" device=""/>
-<part name="SUPPLY22" library="supply2" library_urn="urn:adsk.eagle:library:372" deviceset="+5V" device=""/>
-<part name="+3V6" library="supply1" library_urn="urn:adsk.eagle:library:371" deviceset="+3V3" device=""/>
 <part name="SJ1" library="jumper" library_urn="urn:adsk.eagle:library:252" deviceset="SJ" device="" package3d_urn="urn:adsk.eagle:package:15471/1"/>
 <part name="+3V4" library="supply1" library_urn="urn:adsk.eagle:library:371" deviceset="+3V3" device=""/>
@@
 <instance part="L2" gate="A" x="20.32" y="15.24"/>
 <instance part="R6" gate="G$1" x="48.26" y="15.24"/>
-<instance part="JP2" gate="G$1" x="-86.36" y="104.14"/>
-<instance part="JP3" gate="G$1" x="-76.2" y="104.14"/>
-<instance part="JP4" gate="G$1" x="-66.04" y="104.14"/>
-<instance part="SUPPLY20" gate="1" x="-96.52" y="111.76"/>
-<instance part="GND23" gate="1" x="-96.52" y="99.06"/>
-<instance part="JP5" gate="G$1" x="-48.26" y="104.14"/>
-<instance part="JP6" gate="G$1" x="-38.1" y="104.14"/>
-<instance part="JP7" gate="G$1" x="-27.94" y="104.14"/>
-<instance part="GND24" gate="1" x="-58.42" y="99.06"/>
-<instance part="JP8" gate="G$1" x="-10.16" y="104.14"/>
-<instance part="JP9" gate="G$1" x="0" y="104.14"/>
-<instance part="JP10" gate="G$1" x="10.16" y="104.14"/>
-<instance part="GND26" gate="1" x="-20.32" y="99.06"/>
-<instance part="SUPPLY22" gate="+5V" x="-58.42" y="111.76"/>
-<instance part="+3V6" gate="G$1" x="-20.32" y="111.76"/>
 </instances>
 <busses>
@@
 <pinref part="GND18" gate="1" pin="GND"/>
 </segment>
-<segment>
-<pinref part="JP3" gate="G$1" pin="2"/>
-<pinref part="JP4" gate="G$1" pin="2"/>
-<wire x1="-78.74" y1="104.14" x2="-68.58" y2="104.14" width="0.1524" layer="91"/>
-<pinref part="JP2" gate="G$1" pin="2"/>
-<wire x1="-78.74" y1="104.14" x2="-88.9" y2="104.14" width="0.1524" layer="91"/>
-<junction x="-78.74" y="104.14"/>
-<wire x1="-88.9" y1="104.14" x2="-96.52" y2="104.14" width="0.1524" layer="91"/>
-<junction x="-88.9" y="104.14"/>
-<wire x1="-96.52" y1="104.14" x2="-96.52" y2="101.6" width="0.1524" layer="91"/>
-<pinref part="GND23" gate="1" pin="GND"/>
-</segment>
-<segment>
-<pinref part="JP6" gate="G$1" pin="2"/>
-<pinref part="JP7" gate="G$1" pin="2"/>
-<wire x1="-40.64" y1="104.14" x2="-30.48" y2="104.14" width="0.1524" layer="91"/>
-<pinref part="JP5" gate="G$1" pin="2"/>
-<wire x1="-40.64" y1="104.14" x2="-50.8" y2="104.14" width="0.1524" layer="91"/>
-<junction x="-40.64" y="104.14"/>
-<wire x1="-50.8" y1="104.14" x2="-58.42" y2="104.14" width="0.1524" layer="91"/>
-<junction x="-50.8" y="104.14"/>
-<wire x1="-58.42" y1="104.14" x2="-58.42" y2="101.6" width="0.1524" layer="91"/>
-<pinref part="GND24" gate="1" pin="GND"/>
-</segment>
-<segment>
-<pinref part="JP9" gate="G$1" pin="2"/>
-<pinref part="JP10" gate="G$1" pin="2"/>
-<wire x1="-2.54" y1="104.14" x2="7.62" y2="104.14" width="0.1524" layer="91"/>
-<pinref part="JP8" gate="G$1" pin="2"/>
-<wire x1="-2.54" y1="104.14" x2="-12.7" y2="104.14" width="0.1524" layer="91"/>
-<junction x="-2.54" y="104.14"/>
-<wire x1="-12.7" y1="104.14" x2="-20.32" y2="104.14" width="0.1524" layer="91"/>
-<junction x="-12.7" y="104.14"/>
-<wire x1="-20.32" y1="104.14" x2="-20.32" y2="101.6" width="0.1524" layer="91"/>
-<pinref part="GND26" gate="1" pin="GND"/>
-</segment>
 </net>
 <net name="V+" class="0">
@@
 <wire x1="-86.36" y1="-12.7" x2="-86.36" y2="-15.24" width="0.1524" layer="91"/>
 </segment>
-<segment>
-<pinref part="SUPPLY20" gate="1" pin="V+"/>
-<wire x1="-96.52" y1="109.22" x2="-96.52" y2="106.68" width="0.1524" layer="91"/>
-<pinref part="JP2" gate="G$1" pin="1"/>
-<pinref part="JP3" gate="G$1" pin="1"/>
-<wire x1="-88.9" y1="106.68" x2="-78.74" y2="106.68" width="0.1524" layer="91"/>
-<pinref part="JP4" gate="G$1" pin="1"/>
-<wire x1="-78.74" y1="106.68" x2="-68.58" y2="106.68" width="0.1524" layer="91"/>
-<junction x="-78.74" y="106.68"/>
-<wire x1="-88.9" y1="106.68" x2="-96.52" y2="106.68" width="0.1524" layer="91"/>
-<junction x="-88.9" y="106.68"/>
-</segment>
 </net>
 <net name="+5V" class="0">
@@
 <pinref part="C2" gate="G$1" pin="1"/>
 <wire x1="66.04" y1="55.88" x2="66.04" y2="58.42" width="0.1524" layer="91"/>
-</segment>
-<segment>
-<wire x1="-58.42" y1="109.22" x2="-58.42" y2="106.68" width="0.1524" layer="91"/>
-<pinref part="JP5" gate="G$1" pin="1"/>
-<pinref part="JP6" gate="G$1" pin="1"/>
-<wire x1="-50.8" y1="106.68" x2="-40.64" y2="106.68" width="0.1524" layer="91"/>
-<pinref part="JP7" gate="G$1" pin="1"/>
-<wire x1="-40.64" y1="106.68" x2="-30.48" y2="106.68" width="0.1524" layer="91"/>
-<junction x="-40.64" y="106.68"/>
-<wire x1="-50.8" y1="106.68" x2="-58.42" y2="106.68" width="0.1524" layer="91"/>
-<junction x="-50.8" y="106.68"/>
-<pinref part="SUPPLY22" gate="+5V" pin="+5V"/>
 </segment>
 </net>
@@
 <wire x1="53.34" y1="15.24" x2="58.42" y2="15.24" width="0.1524" layer="91"/>
 </segment>
-<segment>
-<wire x1="-20.32" y1="109.22" x2="-20.32" y2="106.68" width="0.1524" layer="91"/>
-<pinref part="JP8" gate="G$1" pin="1"/>
-<pinref part="JP9" gate="G$1" pin="1"/>
-<wire x1="-12.7" y1="106.68" x2="-2.54" y2="106.68" width="0.1524" layer="91"/>
-<pinref part="JP10" gate="G$1" pin="1"/>
-<wire x1="-2.54" y1="106.68" x2="7.62" y2="106.68" width="0.1524" layer="91"/>
-<junction x="-2.54" y="106.68"/>
-<wire x1="-12.7" y1="106.68" x2="-20.32" y2="106.68" width="0.1524" layer="91"/>
-<junction x="-12.7" y="106.68"/>
-<pinref part="+3V6" gate="G$1" pin="+3V3"/>
-</segment>
-</net>
+</net>

Commit message: multiple changes
removed inductor,
fixed layout + schematic
Parts:
- removed C1, C2: 100nF, rcl:C-EUC0603
- removed JP11: (no value), pinhead:PINHD-2X3/90
- removed L2: RLB9012-221KL, jonas_bourns:RLB9012-221KL
- added ISP: (no value), pinhead:PINHD-2X3/90
- C4, C5: device resistor:C-EUC0603 -> rcl:C-EUC0603
Connections:
- removed net N$6: C5.2, L2.2, U1.VO
- removed net N$8: R7.2, U6.B3
- new net N$3: R7.2, U6.B4
- net +5V: now also C4.1, C5.1, ISP.2; no longer C1.1, C2.1, JP11.2
- net EXT_SPI_CLK: now also U6.A4; no longer U6.A3
- net EXT_SPI_CS: now also U6.A1; no longer U6.A4
- net EXT_SPI_MISO: now also U6.A3; no longer U6.A2
- net EXT_SPI_MOSI: now also U6.A2; no longer U6.A1
- net GND: now also C5.2, ISP.6; no longer C1.2, C2.2, C5.1, JP11.6
- net MISO_5V: now also ISP.1; no longer JP11.1
- net MOSI_5V: now also ISP.4; no longer JP11.4
- net N$1: now also R8.2, U6.B3; no longer R9.2, U6.B1
- net N$2: now also R9.2; no longer R8.2
- net RESET: now also ISP.5; no longer JP11.5
- net SCK_5V: now also ISP.3; no longer JP11.3
- net SENSE+3V3: now also U1.VO; no longer C4.1, L2.1
- net SS_5V: now also U6.B1; no longer U6.B4
Other:
- note added: "3.3V Regler"
- note added: "ESC Ausgang"
- note removed: "+3V3"

Commit message: various changes
moved smd components on metric grid
silkscreen, reduced fuckup in part sizes
added output
Parts:
- removed C8, C9: 22pF, rcl:C-EUC0603
- removed R30: 10k, rcl:R-EU_R1206
- removed R32: 1k, rcl:R-EU_R1206
- removed U$1: D24V50F5, niklas_pololu:D24V50F5
- added A1: D24V50F5SINGLESCREW, jonas_pololu:D24V50F5SINGLESCREW
- added C1, C2: 100nF, resistor:C-EUC0603
- added JP2: (no value), pinhead:PINHD-2X8
- added JP3, JP4, JP5, JP6, JP7: (no value), pinhead:PINHD-1X2
- added R10, R11: 4,7k, resistor:R-EU_R0603
- C3: value 0,1µF -> 22pF; device rcl:C-EUC0603 -> resistor:C-EUC0603
- C4: value 100nF -> 22pF; device rcl:C-EUC0603 -> resistor:C-EUC0603
- C5: value 100nF -> 0,1µF; device rcl:C-EUC0603 -> resistor:C-EUC0603
- C6, C7: device rcl:C-EUC0603 -> resistor:C-EUC0603
- JP1: device pinhead:PINHD-2X8 -> pinhead:PINHD-1X2
- Q1: value 20MHz -> IRFR5305PBF; device crystal:CRYSTALHC49UP -> transistor-power:IRFR5305
- Q3: value IRFR5305PBF -> 20MHz; device transistor-power:IRFR5305 -> crystal:CRYSTALHC49UP
- R1: value 1,2k -> 1k; device rcl:R-EU_R0805 -> resistor:R-EU_R0603
- R2: value 250 -> 10k; device rcl:R-EU_R0805 -> resistor:R-EU_R0603
- R3: value 100 -> 2m; device rcl:R-EU_R0805 -> jonas_resistor:CSS2H-3920
- R5: value 2m -> CRA2512-FZ-R040ELF; device jonas_resistor:CSS2H-3920 -> jonas_bourns:CRA2512-FZ-R040ELF
- R6: value CRA2512-FZ-R040ELF -> 1,2k; device jonas_bourns:CRA2512-FZ-R040ELF -> resistor:R-EU_R0603
- R7: value 4,7k -> 250; device rcl:R-EU_R0805 -> resistor:R-EU_R0603
- R8: value 4,7k -> 100; device rcl:R-EU_R0805 -> resistor:R-EU_R0603
- R9: device rcl:R-EU_R0805 -> resistor:R-EU_R0603
- U2: value LTC2946CMSPBF -> TXB0104; device niklas_lt:LTC2946CMSPBF -> SparkFun-IC-Comms:TXB0104PWR
- U3: value LTC2946CMSPBF -> ATMEGA48-20AU; device niklas_lt:LTC2946CMSPBF -> niklas_atmel:ATMEGA48-20AU
- U5: value ATMEGA48-20AU -> LTC2946CMSPBF; device niklas_atmel:ATMEGA48-20AU -> niklas_lt:LTC2946CMSPBF
- U6: value TXB0104 -> LTC2946CMSPBF; device SparkFun-IC-Comms:TXB0104PWR -> niklas_lt:LTC2946CMSPBF
- renumbered D4 to D1, ESC to J1, LED1 to LED_BAT, LED2 to LED_5V, LED3 to LED_3V
Connections:
- net !ALERT_3V3: now also U3A.PC2_(ADC2/PCINT10), U6.GPIO3; no longer U4.GPIO3, U5A.PC2_(ADC2/PCINT10)
- net !ALERT_5V: now also U3A.PC1_(ADC1/PCINT9), U5.GPIO3; no longer U3.GPIO3, U5A.PC1_(ADC1/PCINT9)
- net !ALERT_V+: now also U3A.PC0_(ADC0/PCINT8), U4.GPIO3; no longer U2.GPIO3, U5A.PC0_(ADC0/PCINT8)
- net +3V3: now also JP6.1, JP7.1, R5.2, R8.2, U6.SENSE-; no longer R3.2, R6.2, U4.SENSE-
- net +5V: now also C1.1, C2.1, JP2.1, JP4.1, JP5.1, R4.2, R7.2, U2.VCCB, U3B.AVCC, U3B.VCC, U3B.VCC_2, U5.SENSE-; no longer C4.1, C5.1, JP1.1, R2.2, R5.2, U3.SENSE-, U5B.AVCC, U5B.VCC, U5B.VCC_2, U6.VCCB
- net AKKU-ZWISCHEN: now also Q1.S, R2.2; no longer Q3.S, R30.2
- net BAT_IN: now also Q1.D; no longer Q2.D
- net EXT_!RST: now also JP2.16; no longer JP1.16
- net EXT_3V3: now also JP2.3, U2.VCCA; no longer JP1.3, U6.VCCA
- net EXT_A0: now also JP2.9; no longer JP1.9
- net EXT_A3: now also JP2.7; no longer JP1.7
- net EXT_A4: now also JP2.5; no longer JP1.5
- net EXT_D1: now also JP2.14; no longer JP1.14
- net EXT_D2: now also JP2.12; no longer JP1.12
- net EXT_D9: now also JP2.10; no longer JP1.10
- net EXT_SCL_5V: now also JP2.13; no longer JP1.13
- net EXT_SDA_5V: now also JP2.15; no longer JP1.15
- net EXT_SPI_CLK: now also JP2.11, U2.A4; no longer JP1.11, U6.A4
- net EXT_SPI_CS: now also JP2.8, U2.A1; no longer JP1.8, U6.A1
- net EXT_SPI_MISO: now also JP2.4, U2.A3; no longer JP1.4, U6.A3
- net EXT_SPI_MOSI: now also JP2.6, U2.A2; no longer JP1.6, U6.A2
- net GND: now also A1.GND, C1.2, C2.2, JP2.2, JP3.2, JP4.2, JP5.2, JP6.2, JP7.2, R1.1, U3B.GND, U3B.GND_2, U3B.GND_3, U4.ADR0, U4.ADR1, U5.ADR0, U5.GND; no longer C8.2, C9.2, R32.1, U$1.GND, U2.ADR0, U2.ADR1, U3.ADR0, U3.GND, U5B.GND, U5B.GND_2, U5B.GND_3
- net GPIO1_3V3: now also U6.GPIO1; no longer U4.GPIO1
- net GPIO1_5V: now also U5.GPIO1; no longer U3.GPIO1
- net GPIO1_V+: now also U4.GPIO1; no longer U2.GPIO1
- net GPIO2_3V3: now also U6.GPIO2; no longer U4.GPIO2
- net GPIO2_5V: now also U5.GPIO2; no longer U3.GPIO2
- net GPIO2_V+: now also U4.GPIO2; no longer U2.GPIO2
- net INTVCC_3V3: now also U6.ADR0, U6.ADR1, U6.INTVCC; no longer U4.ADR0, U4.ADR1, U4.INTVCC
- net INTVCC_5V: now also U5.ADR1, U5.INTVCC; no longer U3.ADR1, U3.INTVCC
- net INTVCC_V+: now also C5.1, U4.INTVCC; no longer C3.1, U2.INTVCC
- net MISO_5V: now also R10.1, U3A.(PCINT4/MISO)_PB4; no longer R8.1, U5A.(PCINT4/MISO)_PB4
- net MOSI_5V: now also U3A.(PCINT3/OC2A/MOSI)_PB3; no longer U5A.(PCINT3/OC2A/MOSI)_PB3
- net N$1: now also R10.2, U2.B3; no longer R8.2, U6.B3
- net N$2: now also U2.B2; no longer U6.B2
- net N$27: now also C3.1, Q3.2, U3A.(PCINT6/XTAL1/TOSC1)_PB6; no longer C8.1, Q1.2, U5A.(PCINT6/XTAL1/TOSC1)_PB6
- net N$28: now also C4.1, Q3.1, U3A.(PCINT7/XTAL2/TOSC2)_PB7; no longer C9.1, Q1.1, U5A.(PCINT7/XTAL2/TOSC2)_PB7
- net N$3: now also R11.2, U2.B4; no longer R7.2, U6.B4
- net N$4: now also R6.1; no longer R1.1
- net N$41: now also Q1.G, R1.2, R2.1; no longer Q3.G, R30.1, R32.2
- net N$5: now also R7.1; no longer R2.1
- net N$7: now also R8.1; no longer R3.1
- net RESET: now also U3A.PC6_(RESET/PCINT14); no longer U5A.PC6_(RESET/PCINT14)
- net SCK_5V: now also R11.1, U3A.PB5_(SCK/PCINT5); no longer R7.1, U5A.PB5_(SCK/PCINT5)
- net SCL: now also U3A.PC5_(ADC5/SCL/PCINT13), U5.SCL, U6.SCL; no longer U2.SCL, U3.SCL, U5A.PC5_(ADC5/SCL/PCINT13)
- net SDA: now also U3A.PC4_(ADC4/SDA/PCINT12), U5.SDAI, U5.SDAO, U6.SDAI, U6.SDAO; no longer U2.SDAI, U2.SDAO, U3.SDAI, U3.SDAO, U5A.PC4_(ADC4/SDA/PCINT12)
- net SENSE+3V3: now also R5.1, U6.SENSE+; no longer R6.1, U4.SENSE+
- net SENSE+5V: now also A1.VOUT, R4.1, U5.SENSE+; no longer R5.1, U$1.VOUT, U3.SENSE+
- net SENSE+V+: now also Q2.D, R3.1, U4.SENSE+; no longer Q3.D, R4.1, U2.SENSE+
- net SS_5V: now also U2.B1, U3A.(PCINT2/SS!/OC1B)_PB2; no longer U5A.(PCINT2/SS!/OC1B)_PB2, U6.B1
- net V+: now also A1.VIN, JP1.1, JP3.1, R3.2, R6.2, U4.SENSE-, U5.VDD, U6.VDD; no longer R1.2, R4.2, U$1.VIN, U2.SENSE-, U2.VDD, U3.VDD
