File: PDB.sch (KiCad schematic (older format))
At the start: 3 parts

Commit message: fix footprints
Parts:
- R? (x2): footprint (none) -> Resistor_SMD:R_0603_1608Metric
Changed lines of the file:
@@
 F 0 "R?" V 8600 2250 50  0000 C CNN
 F 1 "10k" H 8659 2205 50  0001 L CNN
-F 2 "" H 8600 2250 50  0001 C CNN
+F 2 "Resistor_SMD:R_0603_1608Metric" H 8600 2250 50  0001 C CNN
 F 3 "~" H 8600 2250 50  0001 C CNN
 	1    8600 2250
@@
 F 0 "R?" V 8700 2250 50  0000 C CNN
 F 1 "10k" H 8750 2250 50  0000 L CNN
-F 2 "" H 8700 2250 50  0001 C CNN
+F 2 "Resistor_SMD:R_0603_1608Metric" H 8700 2250 50  0001 C CNN
 F 3 "~" H 8700 2250 50  0001 C CNN
 	1    8700 2250
