File: FT230.sch (KiCad schematic (older format))
At the start: 15 parts

Commit message: fix footprints
Parts:
- removed U?: FT230XQ, Package_DFN_QFN:QFN-16-1EP_4x4mm_P0.65mm_EP2.5x2.5mm, symbol Interface_USB:FT230XQ
- added U?: FT230XQ, Package_DFN_QFN:QFN-16-1EP_4x4mm_P0.65mm_EP2.1x2.1mm, symbol Interface_USB:FT230XQ
- C? (x2): footprint (none) -> Capacitor_SMD:C_0603_1608Metric
- D? (x2): footprint (none) -> LED_SMD:LED_0603_1608Metric
- J?: footprint (none) -> GT-USB-7010:USB_C_Receptacle_GT-USB-7010
- R? (x7): footprint (none) -> Resistor_SMD:R_0603_1608Metric
- R?: value R_Small -> 27; footprint (none) -> Resistor_SMD:R_0603_1608Metric
- U?: footprint (none) -> Housings_SOIC:SOIC-8_3.9x4.9mm_Pitch1.27mm
Connections:
- net GNDS: now also U?.13 (GND), U?.17 (GND), U?.3 (GND)
- net at R?.1, R?.1, R?.1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: now also U?.1 (VCCIO), U?.8 (3V3OUT)
- net at J?.A4 (VBUS), J?.A9 (VBUS), J?.B4 (VBUS)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: now also U?.10 (VCC)
- net at D?.1 (K): now also U?.11 (CBUS1)
- net at R?.2, U?.2 (A1): now also U?.15 (TXD)
- net at R?.2, U?.3 (A2): now also U?.2 (RXD)
- net at D?.1 (K): now also U?.5 (CBUS2)
- net at C?.1, R?.1: now also U?.6 (USBDP)
- net at C?.1, R?.1: now also U?.7 (USBDM)
Changed lines of the file:
@@
 $EndDescr
-$Comp
-L Interface_USB:FT230XQ U?
-U 1 1 5C2E33A2
-P 4500 2850
-F 0 "U?" H 4500 3728 50  0000 C CNN
-F 1 "FT230XQ" H 4500 3637 50  0000 C CNN
-F 2 "Package_DFN_QFN:QFN-16-1EP_4x4mm_P0.65mm_EP2.5x2.5mm" H 5050 2150 50  0001 C CNN
-F 3 "http://www.ftdichip.com/Products/ICs/FT230X.html" H 4500 2850 50  0001 C CNN
-	1    4500 2850
-	1    0    0    -1
-$EndComp
 $Comp
 L Connector:USB_C_Receptacle_USB2.0 J?
@@
 F 0 "J?" H 2455 3617 50  0000 C CNN
 F 1 "USB_C_Receptacle_USB2.0" H 2455 3526 50  0000 C CNN
-F 2 "" H 2500 2750 50  0001 C CNN
+F 2 "GT-USB-7010:USB_C_Receptacle_GT-USB-7010" H 2500 2750 50  0001 C CNN
 F 3 "https://www.usb.org/sites/default/files/documents/usb_type-c.zip" H 2500 2750 50  0001 C CNN
 	1    2350 2750
@@
 F 0 "R?" V 3150 2450 50  0000 C CNN
 F 1 "5.1k" V 3045 2450 50  0001 C CNN
-F 2 "" H 3150 2450 50  0001 C CNN
+F 2 "Resistor_SMD:R_0603_1608Metric" H 3150 2450 50  0001 C CNN
 F 3 "~" H 3150 2450 50  0001 C CNN
 F 4 "20%" V 3150 2450 50  0001 C CNN "Tolerance"
@@
 F 0 "R?" V 3150 2350 50  0000 C CNN
 F 1 "5.1k" V 3045 2350 50  0000 C CNN
-F 2 "" H 3150 2350 50  0001 C CNN
+F 2 "Resistor_SMD:R_0603_1608Metric" H 3150 2350 50  0001 C CNN
 F 3 "~" H 3150 2350 50  0001 C CNN
 F 4 "20%" V 3150 2350 50  0001 C CNN "Tolerance"
@@
 F 0 "R?" V 3150 2750 50  0000 C CNN
 F 1 "27" V 3050 2750 50  0000 C CNN
-F 2 "" H 3150 2750 50  0001 C CNN
+F 2 "Resistor_SMD:R_0603_1608Metric" H 3150 2750 50  0001 C CNN
 F 3 "~" H 3150 2750 50  0001 C CNN
 	1    3150 2750
@@
 P 3150 2850
 F 0 "R?" V 3150 2850 50  0000 C CNN
-F 1 "R_Small" V 3050 2850 50  0001 C CNN
-F 2 "" H 3150 2850 50  0001 C CNN
+F 1 "27" V 3050 2850 50  0001 C CNN
+F 2 "Resistor_SMD:R_0603_1608Metric" H 3150 2850 50  0001 C CNN
 F 3 "~" H 3150 2850 50  0001 C CNN
 	1    3150 2850
@@
 F 0 "C?" H 3350 3050 50  0000 L BNN
 F 1 "47p" H 3200 3000 50  0000 R CNN
-F 2 "" H 3300 3000 50  0001 C CNN
+F 2 "Capacitor_SMD:C_0603_1608Metric" H 3300 3000 50  0001 C CNN
 F 3 "~" H 3300 3000 50  0001 C CNN
 	1    3300 3000
@@
 F 0 "C?" H 3500 3050 50  0000 L BNN
 F 1 "47p" H 3542 2955 50  0001 L CNN
-F 2 "" H 3450 3000 50  0001 C CNN
+F 2 "Capacitor_SMD:C_0603_1608Metric" H 3450 3000 50  0001 C CNN
 F 3 "~" H 3450 3000 50  0001 C CNN
 	1    3450 3000
@@
 F 0 "D?" H 5450 3050 50  0000 L BNN
 F 1 "LED_Small" H 5400 3194 50  0001 C CNN
-F 2 "" V 5400 3050 50  0001 C CNN
+F 2 "LED_SMD:LED_0603_1608Metric" V 5400 3050 50  0001 C CNN
 F 3 "~" V 5400 3050 50  0001 C CNN
 	1    5400 3050
@@
 F 0 "R?" V 5700 3050 50  0000 C CNN
 F 1 "270" V 5595 3050 50  0000 C CNN
-F 2 "" H 5700 3050 50  0001 C CNN
+F 2 "Resistor_SMD:R_0603_1608Metric" H 5700 3050 50  0001 C CNN
 F 3 "~" H 5700 3050 50  0001 C CNN
 	1    5700 3050
@@
 F 0 "D?" H 5450 3150 50  0000 L BNN
 F 1 "LED_Small" H 5400 3294 50  0001 C CNN
-F 2 "" V 5400 3150 50  0001 C CNN
+F 2 "LED_SMD:LED_0603_1608Metric" V 5400 3150 50  0001 C CNN
 F 3 "~" V 5400 3150 50  0001 C CNN
 	1    5400 3150
@@
 F 0 "R?" V 5700 3150 50  0000 C CNN
 F 1 "270" V 5595 3150 50  0001 C CNN
-F 2 "" H 5700 3150 50  0001 C CNN
+F 2 "Resistor_SMD:R_0603_1608Metric" H 5700 3150 50  0001 C CNN
 F 3 "~" H 5700 3150 50  0001 C CNN
 	1    5700 3150
@@
 Wire Wire Line
 	4600 2150 4600 2050
-Connection ~ 4600 2150
 Wire Wire Line
 	4600 2150 5300 2150
@@
 F 0 "U?" H 6775 2915 50  0000 C CNN
 F 1 "Si8621" H 6775 2824 50  0000 C CNN
-F 2 "" H 6800 2500 50  0001 C CNN
+F 2 "Housings_SOIC:SOIC-8_3.9x4.9mm_Pitch1.27mm" H 6800 2500 50  0001 C CNN
 F 3 "" H 6800 2500 50  0001 C CNN
 	1    6800 2500
@@
 F 0 "R?" V 5300 2300 50  0000 C CNN
 F 1 "4.7k" H 5250 2300 50  0000 R CNN
-F 2 "" H 5300 2300 50  0001 C CNN
+F 2 "Resistor_SMD:R_0603_1608Metric" H 5300 2300 50  0001 C CNN
 F 3 "~" H 5300 2300 50  0001 C CNN
 	1    5300 2300
@@
 F 0 "R?" V 5450 2300 50  0000 C CNN
 F 1 "4.7k" H 5400 2300 50  0001 R CNN
-F 2 "" H 5450 2300 50  0001 C CNN
+F 2 "Resistor_SMD:R_0603_1608Metric" H 5450 2300 50  0001 C CNN
 F 3 "~" H 5450 2300 50  0001 C CNN
 	1    5450 2300
@@
 Wire Wire Line
 	2050 3700 2350 3700
+$Comp
+L Interface_USB:FT230XQ U?
+U 1 1 5C71DB90
+P 4500 2850
+F 0 "U?" H 4500 3728 50  0000 C CNN
+F 1 "FT230XQ" H 4500 3637 50  0000 C CNN
+F 2 "Package_DFN_QFN:QFN-16-1EP_4x4mm_P0.65mm_EP2.1x2.1mm" H 5050 2150 50  0001 C CNN
+F 3 "http://www.ftdichip.com/Products/ICs/FT230X.html" H 4500 2850 50  0001 C CNN
+	1    4500 2850
+	1    0    0    -1
+$EndComp
+Connection ~ 4600 2150
 $EndSCHEMATC

Commit message: update footprints
Parts:
- U?: footprint Housings_SOIC:SOIC-8_3.9x4.9mm_Pitch1.27mm -> Package_SO:SOIC-8_3.9x4.9mm_P1.27mm
Changed lines of the file:
@@
 encoding utf-8
 Sheet 6 6
-Title ""
-Date ""
+Title "Isolated FT230 USB to UART"
+Date "2019-02-27"
 Rev ""
-Comp ""
+Comp "Toolbox Bodensee e.V."
 Comment1 ""
 Comment2 ""
@@
 F 0 "U?" H 6775 2915 50  0000 C CNN
 F 1 "Si8621" H 6775 2824 50  0000 C CNN
-F 2 "Housings_SOIC:SOIC-8_3.9x4.9mm_Pitch1.27mm" H 6800 2500 50  0001 C CNN
+F 2 "Package_SO:SOIC-8_3.9x4.9mm_P1.27mm" H 6800 2500 50  0001 C CNN
 F 3 "" H 6800 2500 50  0001 C CNN
 	1    6800 2500
