File: PDB.kicad_pcb (KiCad board)
At the start: 2 copper layers, 50 x 80 mm, 95 parts, among them J1 Conn_01x02, J10 Conn_01x02_MountingPin, J11 USB_C_Receptacle_USB2.0, J2 Conn_01x02, J3 Conn_01x02, J4 Conn_01x02, J5 Conn_01x02, J6 Conn_01x02, J7 Conn_01x02, J8 Conn_01x02, J9 Conn_02x03_Odd_Even, SW1 SW_Push, U1 ATmega2560-16AU, U2 LMZM23600, U3 LTC2946, U4 FT230XQ, U5 LMZ13608, U6 LTC2946, Y1 16MHz

Commit message: add large toolbox logo on bottom side
Parts:
- added REF**: ToolboxLogo_Large, Toolbox:ToolboxLogo_Large, B.Cu at (-25.0, 55.0)
Changed lines of the file:
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@@
     (tracks 552)
     (zones 0)
-    (modules 95)
+    (modules 96)
     (nets 54)
   )
@@
     (add_net VBUS)
   )
+  (module Toolbox:ToolboxLogo_Large (layer B.Cu)
+    (at -25 55 180)
+    (fp_text reference REF** (at -0.145 -0.43 180) (layer B.SilkS)
+      (effects (font (size 1 1) (thickness 0.15)) (justify mirror))
+    )
+    (fp_text value ToolboxLogo_Large (at -0.145 0.57 180) (layer B.Fab)
+      (effects (font (size 1 1) (thickness 0.15)) (justify mirror))
+    )
+    (fp_poly (pts (xy -0.00721 18.70819) (xy 16.003384 9.463778) (xy 16.003384 1.881481) (xy 12.675694 -0.001717)
+      (xy 16.003384 -1.886) (xy 16.003384 -9.357199) (xy -0.07 -18.65) (xy -16.080595 -9.419905)
+      (xy -16.080595 9.416497) (xy -12.752903 7.469481) (xy -12.752903 -7.474) (xy -1.765238 -13.815507)
+      (xy -1.765238 -0.88061) (xy -4.402278 -2.387624) (xy -7.72997 -0.441719) (xy 2.25311 5.335484)
+      (xy 5.580802 3.388495) (xy 1.625243 1.065294) (xy 1.625243 -13.815507) (xy 12.738479 -7.410209)
+      (xy 12.738479 -3.769199) (xy 9.410788 -1.948707) (xy 6.020308 -3.894611) (xy 6.020308 -0.064424)
+      (xy 12.738479 3.828497) (xy 12.738479 7.469481) (xy -0.00721 14.815288) (xy -12.752903 7.469481)
+      (xy -16.080595 9.416497)) (layer B.SilkS) (width 0.1))
+  )
   (module Capacitor_SMD:C_1206_3216Metric (layer F.Cu)

Commit message: fix LEDs
Parts:
- D1: value LED -> blue
- D2: value LED -> green
- D3: value LED -> orange
- R1: value 470 -> 2.8k
Changed lines of the file:
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@@
-(kicad_pcb (version 20171130) (host pcbnew 5.1.0-060a0da~80~ubuntu18.04.1)
+(kicad_pcb (version 20171130) (host pcbnew 5.1.1)
   (general
     (thickness 1.6)
@@
       (effects (font (size 1 1) (thickness 0.15)))
     )
-    (fp_text value 470 (at 0 1.43 180) (layer F.Fab)
+    (fp_text value 2.8k (at 0 1.43 180) (layer F.Fab)
       (effects (font (size 1 1) (thickness 0.15)))
     )
@@
       (effects (font (size 1 1) (thickness 0.15)))
     )
-    (fp_text value LED (at 0 1.43) (layer F.Fab)
+    (fp_text value orange (at 0 1.43) (layer F.Fab)
       (effects (font (size 1 1) (thickness 0.15)))
     )
@@
       (effects (font (size 1 1) (thickness 0.15)))
     )
-    (fp_text value LED (at 0 1.43) (layer F.Fab)
+    (fp_text value green (at 0 1.43) (layer F.Fab)
       (effects (font (size 1 1) (thickness 0.15)))
     )
@@
       (effects (font (size 1 1) (thickness 0.15)))
     )
-    (fp_text value LED (at 0 1.43) (layer F.Fab)
-      (effects (font (size 1 1) (thickness 0.15)))
-    )
+    (fp_text value blue (at 0 1.43) (layer F.Fab)
+      (effects (font (size 1 1) (thickness 0.15)))
+    )

Commit message: fix debug LED resistors
Parts:
- R10, R11, R12, R13, R6, R7, R8, R9: value 5.6 -> 100
Changed lines of the file:
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@@
       (effects (font (size 1 1) (thickness 0.15)))
     )
-    (fp_text value 5.6 (at 0 1.43 270) (layer F.Fab)
+    (fp_text value 100 (at 0 1.43 270) (layer F.Fab)
       (effects (font (size 1 1) (thickness 0.15)))
     )
@@
       (effects (font (size 1 1) (thickness 0.15)))
     )
-    (fp_text value 5.6 (at 0 1.43 270) (layer F.Fab)
+    (fp_text value 100 (at 0 1.43 270) (layer F.Fab)
       (effects (font (size 1 1) (thickness 0.15)))
     )
@@
       (effects (font (size 1 1) (thickness 0.15)))
     )
-    (fp_text value 5.6 (at 0 1.43 270) (layer F.Fab)
+    (fp_text value 100 (at 0 1.43 270) (layer F.Fab)
       (effects (font (size 1 1) (thickness 0.15)))
     )
@@
       (effects (font (size 1 1) (thickness 0.15)))
     )
-    (fp_text value 5.6 (at 0 1.43 270) (layer F.Fab)
+    (fp_text value 100 (at 0 1.43 270) (layer F.Fab)
       (effects (font (size 1 1) (thickness 0.15)))
     )
@@
       (effects (font (size 1 1) (thickness 0.15)))
     )
-    (fp_text value 5.6 (at 0 1.43 270) (layer F.Fab)
+    (fp_text value 100 (at 0 1.43 270) (layer F.Fab)
       (effects (font (size 1 1) (thickness 0.15)))
     )
@@
       (effects (font (size 1 1) (thickness 0.15)))
     )
-    (fp_text value 5.6 (at 0 1.43 270) (layer F.Fab)
+    (fp_text value 100 (at 0 1.43 270) (layer F.Fab)
       (effects (font (size 1 1) (thickness 0.15)))
     )
@@
       (effects (font (size 1 1) (thickness 0.15)))
     )
-    (fp_text value 5.6 (at 0 1.43 270) (layer F.Fab)
+    (fp_text value 100 (at 0 1.43 270) (layer F.Fab)
       (effects (font (size 1 1) (thickness 0.15)))
     )
@@
       (effects (font (size 1 1) (thickness 0.15)))
     )
-    (fp_text value 5.6 (at 0 1.43 270) (layer F.Fab)
-      (effects (font (size 1 1) (thickness 0.15)))
-    )
+    (fp_text value 100 (at 0 1.43 270) (layer F.Fab)
+      (effects (font (size 1 1) (thickness 0.15)))
+    )
